File: Maelstrom Boards/Converter/Converter.sch (EAGLE design)
At the start: 72 parts, among them P1 39-30-06, Q10 FDD4141TO252, Q11 BSS123, Q12 BSS123, Q2 BSS123, Q3 BSS123, Q6 BSS123, Q7 BSS123, Q8 FDD4141TO252, Q9 FDD4141TO252

Commit message: Update Converter Board
Parts:
- removed 10K: (no value), resistor:R-US_R0603
- removed Q10, Q8, Q9: FDD4141TO252, transistor-fet:FDD4141TO252
- removed Q2, Q3, Q6: BSS123, transistor-small-signal:BSS123
- removed R18, R19: 10k, resistor:R-US_R0603
- removed R21, R22: 0, resistor:R-US_M2309
- added C1, C20, C6: 0.1uF, rcl:C-EUC0603
- added Q1, Q16, Q17, Q4, Q5: FDD4141TO252, transistor-fet:FDD4141TO252
- added Q13, Q15, Q18: BSS123, transistor-small-signal:BSS123
- added R17, R31, R32, R33, R34, R35, R36, R37, R6: 10k, resistor:R-US_R0603
Connections:
- removed net N$10: 10K.2, Q8.S, R21.1, R22.1
- removed net N$14: Q10.G, Q6.D, R19.1
- removed net N$8: 10K.1, Q2.D, Q8.G
- removed net N$9: Q3.D, Q9.G, R18.1
- new net N$15: Q13.D, Q4.G, R31.1, R6.1
- new net N$22: Q4.D, R17.2
- new net N$23: C1.2, Q1.G, R6.2
- new net N$24: Q15.D, R32.1, R34.1
- new net N$25: C6.2, Q5.G, R32.2
- new net N$26: R33.2
- new net N$27: Q17.G, Q18.D, R35.1, R37.1
- new net N$28: C20.2, Q16.G, R35.2
- new net N$29: Q17.D, R36.2
- net +12V: now also Q1.S, Q4.S, R31.2; no longer Q10.S, Q9.S, R18.2, R19.2, R21.2
- net +5V: now also Q16.S, Q17.S, Q5.S, R34.2, R37.2; no longer R22.2
- net AGND: now also C1.1, C20.1, C6.1, Q13.S, Q15.S, Q18.S; no longer Q2.S, Q3.S, Q6.S
- net JETSON_ON/OFF: now also Q13.G; no longer Q6.G
- net JETSON_SWITCHED: now also Q1.D, R17.1; no longer Q10.D
- net MOBO_ON/OFF: now also Q15.G; no longer Q3.G
- net MOBO_SWITCHED: now also Q5.D, R33.1; no longer Q9.D
- net PLTA_ON/OFF: now also Q18.G; no longer Q2.G
- net PLTA_SWITCHED: now also Q16.D, R36.1; no longer Q8.D
