File: Maelstrom Boards/Converter/Converter.brd (EAGLE design)
At the start: 101.6 x 101.6 mm, 72 parts, among them P1 39-30-06?, Q10 FDD4141TO252, Q11 BSS123, Q12 BSS123, Q2 BSS123, Q3 BSS123, Q6 BSS123, Q7 BSS123, Q8 FDD4141TO252, Q9 FDD4141TO252

Commit message: Update Converter Board
Parts:
- removed 10K: (no value), resistor:R0603
- removed Q10, Q8, Q9: FDD4141TO252, transistor-fet:TO252
- removed Q2, Q3, Q6: BSS123, transistor-small-signal:SOT23
- removed R18, R19: 10k, resistor:R0603
- removed R21, R22: 0, resistor:M2309
- added C1, C20, C6: 0.1uF, rcl:C0603
- added Q1, Q16, Q17, Q4, Q5: FDD4141TO252, transistor-fet:TO252
- added Q13, Q15, Q18: BSS123, transistor-small-signal:SOT23
- added R17, R31, R32, R33, R34, R35, R36, R37, R6: 10k, resistor:R0603
Connections:
- removed net N$10: 10K.2, Q8.2, R21.1, R22.1
- removed net N$14: Q10.1, Q6.3, R19.1
- removed net N$8: 10K.1, Q2.3, Q8.1
- removed net N$9: Q3.3, Q9.1, R18.1
- new net N$15: Q13.3, Q4.1, R31.1, R6.1
- new net N$22: Q4.3, R17.2
- new net N$23: C1.2, Q1.1, R6.2
- new net N$24: Q15.3, R32.1, R34.1
- new net N$25: C6.2, Q5.1, R32.2
- new net N$26: R33.2
- new net N$27: Q17.1, Q18.3, R35.1, R37.1
- new net N$28: C20.2, Q16.1, R35.2
- new net N$29: Q17.3, R36.2
- net +12V: now also Q1.2, Q4.2, R31.2; no longer Q10.2, Q9.2, R18.2, R19.2, R21.2
- net +5V: now also Q16.2, Q17.2, Q5.2, R34.2, R37.2; no longer R22.2
- net AGND: now also C1.1, C20.1, C6.1, Q13.2, Q15.2, Q18.2; no longer Q2.2, Q3.2, Q6.2
- net JETSON_ON/OFF: now also Q13.1; no longer Q6.1
- net JETSON_SWITCHED: now also Q1.3, R17.1; no longer Q10.3
- net MOBO_ON/OFF: now also Q15.1; no longer Q3.1
- net MOBO_SWITCHED: now also Q5.3, R33.1; no longer Q9.3
- net PLTA_ON/OFF: now also Q18.1; no longer Q2.1
- net PLTA_SWITCHED: now also Q16.3, R36.1; no longer Q8.3
Routing:
- net +12V: track 117.7 -> 70.8 mm
- net N$10: track 25.6 -> 0.00 mm
- net N$9: track 8.70 -> 0.00 mm
- net N$14: track 8.68 -> 0.00 mm
- net PLTA_SWITCHED: track 36.0 -> 28.0 mm
- net N$8: track 6.93 -> 0.00 mm
- net MOBO_ON/OFF: track 129.1 -> 122.9 mm
- net JETSON_ON/OFF: track 106.9 -> 100.8 mm
- net AGND: track 85.7 -> 80.8 mm, vias 30 -> 27
- net PLTA_ON/OFF: track 39.0 -> 34.2 mm
- net JETSON_SWITCHED: track 15.7 -> 12.0 mm
- net +5V: track 101.5 -> 97.9 mm
- net MOBO_SWITCHED: track 9.06 -> 6.01 mm

Commit message: Update Converter Board
Parts:
- moved Q4 148.1 mm to (89.4, 87.5)
- moved R17 144.7 mm to (82.9, 91.1)
- moved R6 138.9 mm to (79.8, 79.8), turned to 180 degrees
- moved C1 138.7 mm to (74.8, 79.4)
- moved R31 132.0 mm to (84.8, 78.4)
- moved Q1 125.3 mm to (76.8, 87.4)
- moved Q13 114.3 mm to (75.4, 75.9), turned to 90 degrees
- moved Q5 50.9 mm to (-36.6, -7.75)
- flipped 1C to the bottom
- flipped 1C1 to the bottom
- flipped 1C2 to the bottom
Routing:
- net MOBO_ON/OFF: track 122.9 -> 29.3 mm
- net JETSON_ON/OFF: track 100.8 -> 31.6 mm
- net +5V: track 97.9 -> 67.6 mm, vias 3 -> 1
- net AGND: track 80.8 -> 101.3 mm, vias 27 -> 31
- net N$15: track 0.00 -> 18.5 mm
- net +3V3: track 286.9 -> 302.0 mm, vias 2 -> 7
- net JETSON_SWITCHED: track 12.0 -> 5.74 mm
- net N$22: track 0.00 -> 6.06 mm
- net 3V3MONITORED: track 10.1 -> 15.2 mm
- net 12VFILTERED: track 15.2 -> 19.0 mm, vias 0 -> 1
- net 5VFILTERED: track 21.3 -> 25.1 mm, vias 0 -> 1
- net 3V3FILTERED: track 20.1 -> 23.8 mm, vias 0 -> 1
- net 5VMONITORED: track 7.06 -> 10.8 mm, vias 0 -> 1
- net N$23: track 0.00 -> 3.41 mm
- net 12VMONITORED: track 5.69 -> 8.98 mm, vias 0 -> 1
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